File: Dalmierz/dalmierz/dalmierz.kicad_sch (KiCad schematic)
At the start: 42 parts, among them IC1 W25Q16JVUXIQ, J1 690-005-298-486, Q1 DMG1012T, U1 RP2040, U2 RT6150B-33GQW, U3 LC709203FQH-01TWG

Commit message: MAIN: dalmierz dodaj BLUETOOTH.
Parts:
- removed X1: ~, symbol X1_12MHZ:12MHz
- added C20: 1u, symbol Device:C
- added C21, C22: 2.2uF, symbol Device:C
- added J4: 4328 URM13, 4328:ADAFRUIT_4328, symbol 4328:4328
- added J5: 4328 LCD I2C, 4328:ADAFRUIT_4328, symbol 4328:4328
- added J6: 4328 TF LUNA, 4328:ADAFRUIT_4328, symbol 4328:4328
- added R1: 1k, symbol Device:R
- added SW1, SW2, SW3, SW4, SW5, SW6: SW_Push, symbol Switch:SW_Push
- added U4: LM2775DSGT, LM2775DSGT:SON50P200X200X80-9N, symbol LM2775DSGT:LM2775DSGT
- added Y1: CSTNE12M0GH5L000R0, CSTNE12M0GH5L000R0:OSC_CSTNE12M0GH5L000R0, symbol CSTNE12M0GH5L000R0:CSTNE12M0GH5L000R0
Connections:
- net +3V3: now also J4.2 (VCC), J5.2 (VCC)
- net GND: now also J2.33, C21.1, C22.2, J4.1 (GND), J4.SH1 (SHIELD), J4.SH2 (SHIELD), J5.1 (GND), J5.SH1 (SHIELD), J5.SH2 (SHIELD), J6.1 (GND), J6.SH1 (SHIELD), J6.SH2 (SHIELD), SW1.2, SW2.2, SW3.2, SW4.2, SW5.2, SW6.2, Y1.GND
- net GPIO2: now also SW1.1
- net GPIO3: now also SW2.1
- net GPIO4: now also SW3.1
- net GPIO5: now also SW4.1
- net GPIO6: now also SW5.1
- net GPIO7: now also SW6.1
- net QSPI_SCLK: now also IC1.6 (CLK)
- net QSPI_SD2: now also IC1.3 (~{WP_}(IO2))
- net QSPI_SD3: now also IC1.7 (~{HOLD_OR_RESET_}(IO3))
- net QSPI_SS: now also IC1.1 (~{CS}), R1.2
- net SCL0: now also J4.4 (SCL), J5.4 (SCL), J6.4 (SCL)
- net SDA0: now also J4.3 (SDA), J5.3 (SDA), J6.3 (SDA)
- net VBUS: now also C21.2, U4.7 (VIN)
- net XIN: now also Y1.IN
- net at C17.1, R14.2: now also Y1.OUT
- net at SW1.1, SW1.2: now also R1.1
- new net: C20.1, U4.3 (C1+)
- new net: C20.2, U4.2 (C1-)
- new net +5V: C22.1, J6.2 (VCC), U4.6 (VOUT)
- no-connect marks 7 -> 10
Other:
- note added: "12MHz"
- note added: "ADC GPIO"
- note added: "BLUETOOTH"
- note added: "BOOTSEL"
- note added: "CON PICO"
- note added: "DEBUG"
- note added: "KONEKTORY"
- note added: "LED"
- note added: "OSCYLATOR"
- note added: "PROGRAMOWANIE"
- note added: "PRZYCISKI"
- note added: "RP2040"
- note added: "ZASILANIE"
- moved on the sheet: BT1, C1, C10, C11, C12, C13, C14, C15, C16, C17, C18, C19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

Commit message: MAIN: pierwsza wersja dalmierz.sch.
Parts:
- added B1: ~, symbol BLE_HM-BT4502:BLE_HM-BT4502
Connections:
- net +3V3: now also B1.7 (VDD)
- net GND: now also U4.8 (GND), U4.9 (TP), B1.2 (GND)
- net GPIO10: no longer U1.13 (GPIO10)
- net GPIO12: no longer U1.15 (GPIO12)
- net GPIO13: no longer U1.16 (GPIO13)
- net GPIO2: no longer SW1.1, U1.4 (GPIO2)
- net GPIO3: no longer SW2.1, U1.5 (GPIO3)
- net GPIO4: no longer SW3.1, U1.6 (GPIO4)
- net GPIO5: no longer SW4.1, U1.7 (GPIO5)
- net GPIO6: no longer SW5.1, U1.8 (GPIO6)
- net GPIO7: no longer SW6.1, U1.9 (GPIO7)
- net GPIO8: no longer U1.11 (GPIO8)
- net GPIO9: no longer U1.12 (GPIO9)
- new net BTN1: SW1.1, U1.4 (GPIO2)
- new net BTN2: SW2.1, U1.5 (GPIO3)
- new net BTN3: SW3.1, U1.6 (GPIO4)
- new net BTN4: SW4.1, U1.7 (GPIO5)
- new net BTN5: SW5.1, U1.8 (GPIO6)
- new net BTN6: SW6.1, U1.9 (GPIO7)
- new net BT_INTERRUPT: U1.13 (GPIO10)
- new net BT_INTERUPT: B1.1 (INT)
- new net BT_LOW_POWER: B1.6 (WAKEUP), U1.11 (GPIO8)
- new net BT_POWER_DOWN: B1.5 (PDN), U1.12 (GPIO9)
- new net UART0_RX: B1.9 (TXD), U1.16 (GPIO13)
- new net UART0_TX: B1.8 (RXD), U1.15 (GPIO12)
- no-connect marks 10 -> 14

Commit message: MAIN: 1 wersja dalmierz sch.
Parts:
- removed R2: 100k, symbol Device:R
- added D3: MBR120VLSFT1G, MBR120VLSFT1G:DIOM3616X98N, symbol MBR120VLSFT1G:MBR120VLSFT1G
- added R4, R8: 10k, symbol Device:R
Connections:
- net +3V3: now also R4.1, R8.2
- net 3V3_EN: no longer U2.7 (PS)
- net SCL0: now also R4.2
- net SDA0: now also R8.1
- net VBUS: now also D3.2; no longer C21.2, U4.7 (VIN)
- new net: C21.2, D3.1, U4.7 (VIN)
- no-connect marks 14 -> 15
Other:
- note added: "Wazne jest aby zachować bliska odleglosc kondensatorow odciagajacych od wejsc"
